File: MOM1/MOM1_SPS1_model/MOM1_model.kicad_pcb (KiCad board)
At the start: 4 copper layers, 203 x 116 mm, 9 parts, among them J1 TE_Eurocard_96pole, J2 5-5530843-4, J3 5-5530843-4, J4 5-5530843-4, J5 5-5530843-4

Commit message: Made plenty of change (see CHANGELOG file)
Parts:
- removed HOLE1, HOLE2, HOLE3, HOLE4: MountingHole_3mm, Mounting_Holes:MountingHole_3mm
- added H1: MountingHole_3mm, MountingHole:MountingHole_3mm, F.Cu at (73.0, 37.0)
- added H2: MountingHole_3mm, MountingHole:MountingHole_3mm, F.Cu at (266.0, 37.0)
- added H3: MountingHole_3mm, MountingHole:MountingHole_3mm, F.Cu at (73.0, 143.0)
- added H4: MountingHole_3mm, MountingHole:MountingHole_3mm, F.Cu at (266.0, 143.0)
- J1: value TE_Eurocard_96pole -> Eurocard_5536475-1_inv; footprint Eurocard_5536475-1:Eurocard_5536475-1_Inv -> Eurocard_5536475-1:Eurocard_5536475-1_inv
- J2, J3, J4, J5: value 5-5530843-4 -> PP1_connector_TE_5-5530843-4; footprint Eurocard:SHDR40W89P485X254_2X20_5740X935X1562P -> TE_5-5530843-4:TE_5-5530843-4
Connections:
- J1 pad a32: +5V -> /FEEDBACK
- J2 pad 3: /GLOBAL_CLK -> /PERIPHERAL_CLK
- J3 pad 3: /GLOBAL_CLK -> /PERIPHERAL_CLK
- J4 pad 3: /GLOBAL_CLK -> /PERIPHERAL_CLK
- J5 pad 3: /GLOBAL_CLK -> /PERIPHERAL_CLK
