File: MOM1/MOM1_basic_model/MOM1_model.kicad_pcb (KiCad board)
At the start: 4 copper layers, 203 x 116 mm, 8 parts, among them J2 5-5530843-4, J3 5-5530843-4, J4 5-5530843-4, J5 5-5530843-4

Commit message: Made plenty of change (see CHANGELOG file)
Parts:
- removed HOLE1, HOLE2, HOLE3, HOLE4: MountingHole_3mm, Mounting_Holes:MountingHole_3mm
- added H1: MountingHole_3mm, MountingHole:MountingHole_3mm, F.Cu at (73.0, 37.0)
- added H2: MountingHole_3mm, MountingHole:MountingHole_3mm, F.Cu at (266.0, 37.0)
- added H3: MountingHole_3mm, MountingHole:MountingHole_3mm, F.Cu at (73.0, 143.0)
- added H4: MountingHole_3mm, MountingHole:MountingHole_3mm, F.Cu at (266.0, 143.0)
- J2, J3, J4, J5: value 5-5530843-4 -> PP1_connector_TE_5-5530843-4; footprint Eurocard:SHDR40W89P485X254_2X20_5740X935X1562P -> TE_5-5530843-4:TE_5-5530843-4
Connections:
- net /GLOBAL_CLK renamed /PERIPHERAL_CLK
